Commit message: shrinked sensornode

File: seneka_ugv_description/urdf/sensornode.urdf.xacro (robot description, xacro)
@@ -10,5 +10,5 @@
     <visual>
       <geometry>
-        <box size="0.75 0.25 0.75"/>
+        <box size="0.1 0.1 0.1"/>
       </geometry>
       <origin rpy="2 2 2" xyz="0 0 0"/>
@@ -17,10 +17,10 @@
     <collision>
       <geometry>
-        <box size="0.75 0.75 0.75"/>
+        <box size="0.1 0.1 0.1"/>
       </geometry>
       <origin rpy="2 2 2" xyz="0 0 0"/>
     </collision>
     <inertial>
-      <mass value="60" />
+      <mass value="0.1" />
       <inertia ixx="1.0" ixy="0.0" ixz="0.0" iyy="1.0" iyz="0.0" izz="1.0"/>
     </inertial>

Commit message: ready for groovy_dev branch of Universal Robot

File: seneka_ugv_description/urdf/sensornode.urdf.xacro (robot description, xacro)
@@ -4,23 +4,23 @@
        xmlns:interface="http://playerstage.sourceforge.net/gazebo/xmlschema/#interface"
        xmlns:xacro="http://playerstage.sourceforge.net/gazebo/xmlschema/#interface"
-       name="sensornode">
+       name="">
   <!-- common stuff -->
   <!--  <include filename="$(find seneka_ugv_description)/urdf/sensornode.gazebo.xacro" /> -->
-  <link name="sensornode_body">
+  <link name="sensornode">
     <visual>
       <geometry>
-        <box size="0.1 0.1 0.1"/>
+        <mesh filename="package://seneka_ugv_description/meshes/sensornode_reduced.dae" scale="0.001 0.001 0.001"/>
       </geometry>
-      <origin rpy="2 2 2" xyz="0 0 0"/>
+      <origin rpy="0 0 0" xyz="0 0 0"/>
       <material name="black"/>
     </visual>
     <collision>
       <geometry>
-        <box size="0.1 0.1 0.1"/>
+        <mesh filename="package://seneka_ugv_description/meshes/sensornode_reduced.dae" scale="0.001 0.001 0.001"/>
       </geometry>
-      <origin rpy="2 2 2" xyz="0 0 0"/>
+      <origin rpy="0 0 0" xyz="0 0 0"/>
     </collision>
     <inertial>
-      <mass value="0.1" />
+      <mass value="3.0" />
       <inertia ixx="1.0" ixy="0.0" ixz="0.0" iyy="1.0" iyz="0.0" izz="1.0"/>
     </inertial>

File: seneka_ugv_description/urdf/ugv_robot.urdf.xacro (robot description, xacro)
@@ -11,8 +11,79 @@
  <!-- ur10 -->
  <include filename="$(find ur_description)/urdf/ur10.urdf.xacro" />
+  <!-- Added connector joint for connecting it with a robot -->
+  <joint name="right_arm_ur10_connector" type="fixed">
+    <parent link="quanjo_body" />
+    <child link = "right_arm_base_link" />
+    <origin xyz="0.615 -0.46 0.87" rpy="0 0.2 0" />
+  </joint>
+  <joint name="left_arm_ur10_connector" type="fixed">
+    <parent link="quanjo_body" />
+    <child link = "left_arm_base_link" />
+    <origin xyz="0.615 0.46 0.87" rpy="0 0.2 0" />
+  </joint>
   <!-- arm -->
-  <xacro:ur10_robot prefix="right_arm_"  parent="quanjo_body" x="0.615" y="-0.46" z="0.87" roll="0" pitch="0.2" yaw="0">
+  <xacro:ur10_robot prefix="right_arm_">
   </xacro:ur10_robot>
-  <xacro:ur10_robot prefix="left_arm_" parent="quanjo_body" x="0.615" y="0.46"  z="0.87" roll="0" pitch="0.2" yaw="0">
+  <xacro:ur10_robot prefix="left_arm_">
   </xacro:ur10_robot>
+  <joint name=" right_arm_gripper_joint" type="fixed">
+    <parent link="right_arm_ee_link" />
+    <child link = "right_arm_gripper_link" />
+    <origin xyz="0.0 0.0 0.0" rpy="0.0 0.0 0.0" />
+  </joint>
+  <link name="right_arm_gripper_link">
+    <visual>
+      <geometry>
+        <mesh filename="package://seneka_ugv_description/meshes/gripper.dae" scale="0.001 0.001 0.001"/>
+      </geometry>
+      <origin xyz="0.0 0.0 0.0" rpy="0.0 -1.57 0.0" />
+    </visual>
+    <collision>
+      <geometry>
+          <mesh filename="package://seneka_ugv_description/meshes/gripper.dae" scale="0.001 0.001 0.001"/>
+      </geometry>
+      <origin xyz="0.0 0.0 0.0" rpy="0.0 -1.57 0.0" />
+    </collision>
+    <inertial>
+      <mass value="1" />
+      <origin xyz="0.0 0.0 0.0" rpy="0.0 0.0 0.0" />
+      <inertia ixx="1.0" ixy="0.0" ixz="0.0" iyy="1.0" iyz="0.0" izz="1.0"/>
+    </inertial>
+  </link>
+   <joint name="right_arm_rviz_joint" type="fixed">
+    <parent link="right_arm_gripper_link" />
+    <child link = "right_arm_rviz_link" />
+    <origin xyz="0.0 0.0 0.0" rpy="0.0 0.0 ${pi/2.0}" />
+  </joint>
+  <link name="right_arm_rviz_link" />
+  <joint name="left_arm_gripper_joint" type="fixed">
+    <parent link="left_arm_ee_link" />
+    <child link = "left_arm_gripper_link" />
+    <origin xyz="0.0 0.0 0.0" rpy="0.0 0.0 0.0" />
+  </joint>
+ <link name="left_arm_gripper_link">
+    <visual>
+      <geometry>
+        <mesh filename="package://seneka_ugv_description/meshes/gripper.dae" scale="0.001 0.001 0.001"/>
+      </geometry>
+      <origin xyz="0.0 0.0 0.0" rpy="0.0 -1.57 0.0" />
+    </visual>
+    <collision>
+      <geometry>
+          <mesh filename="package://seneka_ugv_description/meshes/gripper.dae" scale="0.001 0.001 0.001"/>
+      </geometry>
+      <origin xyz="0.0 0.0 0.0" rpy="0.0 -1.57 0.0" />
+    </collision>
+    <inertial>
+      <mass value="1" />
+      <origin xyz="0.0 0.0 0.0" rpy="0.0 0.0 0.0" />
+      <inertia ixx="1.0" ixy="0.0" ixz="0.0" iyy="1.0" iyz="0.0" izz="1.0"/>
+    </inertial>
+  </link>
+   <joint name="left_arm_rviz_joint" type="fixed">
+    <parent link="left_arm_gripper_link" />
+    <child link = "left_arm_rviz_link" />
+    <origin xyz="0.0 0.0 0.0" rpy="0.0 0.0 ${pi/2.0}" />
+  </joint>
+  <link name="left_arm_rviz_link" />
 </robot>
