Commit message: sensornode detection prepared for gazebo simulation

File: seneka_ugv_description/urdf/sensornode.gazebo.xacro (robot description, xacro)
@@ -3,4 +3,5 @@
        xmlns:controller="http://playerstage.sourceforge.net/gazebo/xmlschema/#controller"
        xmlns:interface="http://playerstage.sourceforge.net/gazebo/xmlschema/#interface">
-<gazebo></gazebo>
+<gazebo>
+</gazebo>
 </robot>

File: seneka_ugv_description/urdf/sensornode.urdf.xacro (robot description, xacro)
@@ -22,7 +22,8 @@
     </collision>
     <inertial>
-      <mass value="3.0" />
+      <mass value="30.0" />
       <inertia ixx="1.0" ixy="0.0" ixz="0.0" iyy="1.0" iyz="0.0" izz="1.0"/>
     </inertial>
   </link>
+  <gravity>false</gravity>
 </robot>

File: seneka_ugv_description/urdf/ugv_robot.urdf.xacro (robot description, xacro)
@@ -87,3 +87,4 @@
   </joint>
   <link name="left_arm_rviz_link" />
+ <gravity>false</gravity>
 </robot>
