Commit message: added sensornode files

File: seneka_ugv_description/urdf/ugv.urdf.xacro (robot description, xacro)
@@ -4,11 +4,12 @@
        xmlns:interface="http://playerstage.sourceforge.net/gazebo/xmlschema/#interface"
        xmlns:xacro="http://ros.org/wiki/xacro">
-   <material name="white">
-  	<color rgba="1 1 1 1"/>
-   </material>
-   <material name="black">
-  	<color rgba="0 0 0 1"/>
-   </material>
-  <link name="ugv_companio_body">
+ <!--  <property name="camera_origin" value=" 0.0 0.0 0.0" /> -->
+  <material name="white">
+    <color rgba="1 1 1 1"/>
+  </material>
+  <material name="black">
+    <color rgba="0 0 0 1"/>
+  </material>
+  <link name="quanjo_body">
     <visual>
       <geometry>
@@ -31,30 +32,3 @@
     </inertial>
   </link>
-<!--  <joint name="neck_joint" type="fixed">
-    <parent link="ugv_companio_body" />
-    <child link ="ugv_companio_head" />
-    <origin xyz="0.0 0.0 1" rpy="0.0 0.0 0.0" />
-    <axis xyz="0.0 0.0 1.0" />
-    <limit lower="0" upper="1" effort="1" velocity="1"/>
-    <dynamics damping="1000" friction="0.1"/>
-  </joint>
-  <link name="ugv_companio_head">
-    <visual>
-      <geometry>
-        <box size=".5 .5 .5"/>
-      </geometry>
-      <origin xyz="0 0 -0.125" rpy="0 0 0"/>
-      <material name="white"/>
-    </visual>
-    <collision>
-      <geometry>
-        <box size=".5 .5 .5"/>
-      </geometry>
-      <origin xyz="0 0 -0.125" rpy="0 0 0"/>
-    </collision>
-    <inertial>
-      <mass value="40" />
-      <inertia ixx="1.0" ixy="0.0" ixz="0.0" iyy="1.0" iyz="0.0" izz="1.0"/>
-    </inertial>
-  </link> -->
 </robot>

File: seneka_ugv_description/urdf/ugv_robot.urdf.xacro (robot description, xacro)
@@ -5,14 +5,14 @@
        xmlns:xacro="http://playerstage.sourceforge.net/gazebo/xmlschema/#interface"
        name="sugv">
-  <!-- common stuff -->
-  <include filename="$(find ur_description)/urdf/gazebo.urdf.xacro" />
- <!-- compagnio description -->
-  <include filename="$(find seneka_ugv_description)/urdf/ugv.urdf.xacro" />
+ <!-- common stuff -->
+ <include filename="$(find ur_description)/urdf/gazebo.urdf.xacro" />
+ <!-- quanjo description -->
+ <include filename="$(find seneka_ugv_description)/urdf/ugv.urdf.xacro" />
  <!-- ur10 -->
-  <include filename="$(find ur_description)/urdf/ur10.urdf.xacro" />
+ <include filename="$(find ur_description)/urdf/ur10.urdf.xacro" />
   <!-- arm -->
-  <xacro:ur10_robot prefix="right_arm_"  parent="ugv_companio_body" x="0.615" y="-0.46" z="0.87" roll="0" pitch="0.2" yaw="0">
+  <xacro:ur10_robot prefix="right_arm_"  parent="quanjo_body" x="0.615" y="-0.46" z="0.87" roll="0" pitch="0.2" yaw="0">
   </xacro:ur10_robot>
-  <xacro:ur10_robot prefix="left_arm_" parent="ugv_companio_body" x="0.615" y="0.46"  z="0.87" roll="0" pitch="0.2" yaw="0">
+  <xacro:ur10_robot prefix="left_arm_" parent="quanjo_body" x="0.615" y="0.46"  z="0.87" roll="0" pitch="0.2" yaw="0">
   </xacro:ur10_robot>
 </robot>

Commit message: arm movement is working

File: seneka_ugv_description/urdf/ugv.urdf.xacro (robot description, xacro)
@@ -11,4 +11,10 @@
     <color rgba="0 0 0 1"/>
   </material>
+  <link name="world_dummy_link"></link>
+  <joint name="world_dummy_joint" type="fixed">
+    <parent link="world_dummy_link" />
+    <child link = "quanjo_body" />
+    <origin xyz="0.0 0.0 0.0" rpy="0.0 0.0 0.0" />
+  </joint>
   <link name="quanjo_body">
     <visual>

File: seneka_ugv_description/urdf/ugv_robot.urdf.xacro (robot description, xacro)
@@ -15,10 +15,10 @@
   <parent link="quanjo_body" />
   <child link = "right_arm_base_link" />
-  <origin xyz="0.615 -0.46 0.87" rpy="0 0.2 0" />
+  <origin xyz="0.615 -0.46 0.87" rpy="-0.2 0 -1.57" />
  </joint>
  <joint name="left_arm_ur10_connector" type="fixed">
   <parent link="quanjo_body" />
   <child link = "left_arm_base_link" />
-  <origin xyz="0.615 0.46 0.87" rpy="0 0.2 0" />
+  <origin xyz="0.615 0.46 0.87" rpy="-0.2 0 -1.57" />
  </joint>
   <!-- arm -->
@@ -37,11 +37,11 @@
         <mesh filename="package://seneka_ugv_description/meshes/gripper.dae" scale="0.001 0.001 0.001"/>
       </geometry>
-      <origin xyz="0.0 0.0 0.0" rpy="0.0 -1.57 0.0" />
+      <origin xyz="0.0 0.0 0.0" rpy="1.57 0 -1.57" />
     </visual>
     <collision>
       <geometry>
-          <mesh filename="package://seneka_ugv_description/meshes/gripper.dae" scale="0.001 0.001 0.001"/>
+          <box size="0.09 0.32 0.05" />
       </geometry>
-      <origin xyz="0.0 0.0 0.0" rpy="0.0 -1.57 0.0" />
+      <origin xyz="0.0 0.0 -0.115" rpy="1.57 0 -1.57" />
     </collision>
     <inertial>
@@ -67,11 +67,11 @@
         <mesh filename="package://seneka_ugv_description/meshes/gripper.dae" scale="0.001 0.001 0.001"/>
       </geometry>
-      <origin xyz="0.0 0.0 0.0" rpy="0.0 -1.57 0.0" />
+        <origin xyz="0.0 0.0 0.0" rpy="1.57 0 -1.57" />
     </visual>
     <collision>
       <geometry>
-          <mesh filename="package://seneka_ugv_description/meshes/gripper.dae" scale="0.001 0.001 0.001"/>
+          <box size="0.09 0.32 0.05" />
       </geometry>
-      <origin xyz="0.0 0.0 0.0" rpy="0.0 -1.57 0.0" />
+      <origin xyz="0.0 0.0 -0.115" rpy="1.57 0 -1.57" />
     </collision>
     <inertial>

Commit message: added state machine in seneka_pnp and services

File: seneka_ugv_description/urdf/ugv.urdf.xacro (robot description, xacro)
@@ -20,6 +20,9 @@
     <visual>
       <geometry>
-        <!-- <box size="0.75 0.75 0.75"/> -->
+        <!--<box size="1.12 1.10 0.55"/>-->
  	<mesh filename="package://seneka_ugv_description/meshes/quanjo_grob.dae" scale="0.001 0.001 0.001"/>
+      </geometry>
+      <geometry>
+      	<box size="0.5 0.5 2.0"/>
       </geometry>
       <origin rpy="0 0 1.57" xyz="0 0 0"/>

Commit message: working on stability of cartesian planner

File: seneka_ugv_description/urdf/ugv.urdf.xacro (robot description, xacro)
@@ -21,5 +21,5 @@
       <geometry>
         <!--<box size="1.12 1.10 0.55"/>-->
- 	<mesh filename="package://seneka_ugv_description/meshes/quanjo_grob.dae" scale="0.001 0.001 0.001"/>
+ 	<mesh filename="package://seneka_ugv_description/meshes/Mockup_simplified.dae" scale="0.001 0.001 0.001"/>
       </geometry>
       <geometry>
@@ -32,5 +32,5 @@
       <geometry>
         <!-- <box size="0.75 0.75 0.75"/> -->
-	<mesh filename="package://seneka_ugv_description/meshes/quanjo_grob.dae" scale="0.001 0.001 0.001"/>
+	<mesh filename="package://seneka_ugv_description/meshes/Mockup_simplified.dae" scale="0.001 0.001 0.001"/>
       </geometry>
       <origin rpy="0 0 1.57" xyz="0 0 0"/>

File: seneka_ugv_description/urdf/ugv_robot.urdf.xacro (robot description, xacro)
@@ -15,4 +15,5 @@
   <parent link="quanjo_body" />
   <child link = "right_arm_base_link" />
+  <!--<origin xyz="0.615 -0.46 0.87" rpy="-0.2 0 -1.57" />-->
   <origin xyz="0.615 -0.46 0.87" rpy="-0.2 0 -1.57" />
  </joint>
@@ -20,4 +21,5 @@
   <parent link="quanjo_body" />
   <child link = "left_arm_base_link" />
+  <!--<origin xyz="0.615 0.46 0.87" rpy="-0.2 0 -1.57" />-->
   <origin xyz="0.615 0.46 0.87" rpy="-0.2 0 -1.57" />
  </joint>
