Commit message: planning works

File: seneka_ugv_description/urdf/ugv_robot.urdf.xacro (robot description, xacro)
@@ -11,15 +11,15 @@
  <!-- ur10 -->
  <include filename="$(find ur_description)/urdf/ur10.urdf.xacro" />
-  <!-- Added connector joint for connecting it with a robot -->
-  <joint name="right_arm_ur10_connector" type="fixed">
-    <parent link="quanjo_body" />
-    <child link = "right_arm_base_link" />
-    <origin xyz="0.615 -0.46 0.87" rpy="0 0.2 0" />
-  </joint>
-  <joint name="left_arm_ur10_connector" type="fixed">
-    <parent link="quanjo_body" />
-    <child link = "left_arm_base_link" />
-    <origin xyz="0.615 0.46 0.87" rpy="0 0.2 0" />
-  </joint>
+ <!-- Added connector joint for connecting it with a robot -->
+ <joint name="right_arm_ur10_connector" type="fixed">
+  <parent link="quanjo_body" />
+  <child link = "right_arm_base_link" />
+  <origin xyz="0.615 -0.46 0.87" rpy="0 0.2 0" />
+ </joint>
+ <joint name="left_arm_ur10_connector" type="fixed">
+  <parent link="quanjo_body" />
+  <child link = "left_arm_base_link" />
+  <origin xyz="0.615 0.46 0.87" rpy="0 0.2 0" />
+ </joint>
   <!-- arm -->
   <xacro:ur10_robot prefix="right_arm_">

Commit message: teach mode added

File: seneka_ugv_description/urdf/ugv_robot.urdf.xacro (robot description, xacro)
@@ -27,5 +27,5 @@
   <xacro:ur10_robot prefix="left_arm_">
   </xacro:ur10_robot>
-  <joint name=" right_arm_gripper_joint" type="fixed">
+  <joint name="right_arm_gripper_joint" type="fixed">
     <parent link="right_arm_ee_link" />
     <child link = "right_arm_gripper_link" />

Commit message: new rear jointstates

File: seneka_ugv_description/urdf/ugv_robot.urdf.xacro (robot description, xacro)
@@ -16,5 +16,5 @@
   <child link = "right_arm_base_link" />
   <!--<origin xyz="0.615 -0.46 0.87" rpy="-0.2 0 -1.57" />-->
-  <origin xyz="0.615 -0.46 0.87" rpy="-0.2 0 -1.57" />
+  <origin xyz="0.53 -0.4775 0.89" rpy="-0.2 0 -1.57" />
  </joint>
  <joint name="left_arm_ur10_connector" type="fixed">
@@ -22,5 +22,5 @@
   <child link = "left_arm_base_link" />
   <!--<origin xyz="0.615 0.46 0.87" rpy="-0.2 0 -1.57" />-->
-  <origin xyz="0.615 0.46 0.87" rpy="-0.2 0 -1.57" />
+  <origin xyz="0.53 0.4775 0.89" rpy="-0.2 0 -1.57" />
  </joint>
   <!-- arm -->
